File: pcb/Braille-Pogo-Frame/Braille-Pogo-Frame.kicad_pcb (KiCad board)
At the start: 2 copper layers, 76 x 95 mm, 64 parts, among them J1 Conn_01x06, J10 Screw_Terminal_01x02, J2 Conn_01x06, J3 Conn_01x06, J4 Conn_01x06, J9 Conn_01x02, M1 Stepper_Motor_bipolar, M2 Stepper_Motor_bipolar, M3 Stepper_Motor_bipolar, M4 Stepper_Motor_bipolar, SW1 SW_Push, SW2 SW_Push, U1 DRV8847SPWR, U2 DRV8847SPWR, U3 DRV8847SPWR, U4 DRV8847SPWR, U9 RP2040-Zero

Commit message: Routing and finishing touches; ready to order
Routing:
- net GND: track 0.00 -> 192.0 mm, vias 0 -> 39
- net Vdrive: track 0.00 -> 166.6 mm, vias 0 -> 2
- net I2C_SDA: track 0.00 -> 150.7 mm
- net I2C_SCL: track 0.00 -> 148.8 mm
- net +3V3: track 0.00 -> 127.6 mm, vias 0 -> 3
- net /Braille_Cell/~{FAULT}: track 0.00 -> 83.4 mm
- net /Braille_Cell1/~{FAULT}: track 0.00 -> 61.6 mm
- net /Braille_Cell2/~{FAULT}: track 0.00 -> 58.1 mm, vias 0 -> 1
- net /Braille_Cell2/~{SLEEP}: track 0.00 -> 57.9 mm, vias 0 -> 1
- net /Braille_Cell/IN1: track 0.00 -> 51.7 mm, vias 0 -> 1
- net /Braille_Cell/IN3: track 0.00 -> 50.5 mm, vias 0 -> 1
- net /Braille_Cell/IN2: track 0.00 -> 50.4 mm, vias 0 -> 1
- net /Braille_Cell/~{SLEEP}: track 0.00 -> 48.4 mm, vias 0 -> 1
- net /Braille_Cell/IN4: track 0.00 -> 46.0 mm, vias 0 -> 1
- net /Braille_Cell3/~{FAULT}: track 0.00 -> 41.9 mm, vias 0 -> 1
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- added copper zone on B.Cu, net GND
- added copper zone on F.Cu, net GND
Other:
- board text added: "Vdr GND"
- board text added: "Vdrive GND"
