File: idea_column_rods/Braille-Column-Rods-PCB/Braille-Column-Rods-PCB.kicad_pcb (KiCad board)
At the start: 2 copper layers, 95 x 99 mm, 156 parts, among them J1 Conn_01x03, J2 Conn_01x02, J3 Conn_01x02, J4 Conn_01x08, J5 Screw_Terminal_01x02, J6 Screw_Terminal_01x02, J7 Conn_01x02, M1 Stepper_Motor_bipolar, M10 Motor_DC_With_MP, M11 Motor_DC_With_MP, M12 Motor_DC_With_MP, M2 Stepper_Motor_bipolar, M3 Stepper_Motor_bipolar, M4 Stepper_Motor_bipolar, M5 Stepper_Motor_bipolar, M6 Stepper_Motor_bipolar, M7 Stepper_Motor_bipolar, M8 Stepper_Motor_bipolar, M9 Motor_DC_With_MP, SW1 SW_Push, SW2 SW_Push, U1 DRV8847SPWR, U10 AD116, U11 AD116, U12 AD116, U13 AD116, U14 74HC595, U15 74HC595, U17 MT910xET, U18 MT910xET, U19 MT910xET, U2 DRV8847SPWR, U20 MT910xET, U21 MT910xET, U22 MT910xET, U23 MT910xET, U24 MT910xET, U25 MT910xET, U26 MT910xET, U27 MT910xET, U28 MT910xET, U3 RP2040-Zero, U30 CD74HC4067M, U4 DRV8847SPWR, U5 DRV8847SPWR, U6 DRV8847SPWR, U7 DRV8847SPWR, U8 DRV8847SPWR, U9 DRV8847SPWR

Commit message: WIP: Manual routing and silkscreens
Parts:
- removed J2: Conn_01x02, Connector_PinHeader_2.54mm:PinHeader_1x02_P2.54mm_Vertical
- moved U15 165.3 mm to (140.0, 132.1)
- moved C15 165.1 mm to (145.6, 127.5)
- moved J7 162.9 mm to (157.2, 116.5), turned to 90 degrees
- moved C14 162.7 mm to (145.8, 114.8)
- moved R43 156.1 mm to (150.2, 109.2)
- moved C43 155.2 mm to (150.2, 97.5)
- moved U14 155.0 mm to (140.0, 119.3)
- moved U30 154.8 mm to (142.4, 104.8)
- moved J5 137.6 mm to (175.0, 98.3), turned to 90 degrees
- moved J6 137.1 mm to (175.0, 109.0), turned to 90 degrees
- moved R17 67.1 mm to (154.5, 121.7), turned to -90 degrees
- moved R18 64.5 mm to (158.2, 121.5), turned to -90 degrees
- moved C9 59.9 mm to (164.0, 102.9)
- moved D3 10.7 mm to (167.2, 108.9), turned to -90 degrees
- moved R3 8.57 mm to (168.1, 111.8), turned to 180 degrees
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Connections:
- C9 pad 1: Vdrive -> VDC
- U3 pad 8: Net-(J2-Pin_1) -> I2C_SCL
- U3 pad 9: Net-(J2-Pin_2) -> I2C_SDA
Routing:
- net +3V3: track 7.64 -> 33.8 mm
- net +5V: track 0.00 -> 18.3 mm
- net /Microcontroller/HALL_ANALOG: track 0.00 -> 11.6 mm
- net /Microcontroller/GP_LED_0: track 0.00 -> 10.7 mm
- net VDC: track 42.0 -> 49.9 mm
- net /Microcontroller/SW_1: track 0.00 -> 6.12 mm
- net /Microcontroller/GP_LED_1: track 0.00 -> 5.54 mm
- net /Microcontroller/SW_2: track 0.00 -> 5.41 mm
- net I2C_SDA: track 0.00 -> 5.10 mm
- net I2C_SCL: track 0.00 -> 4.25 mm
- net Net-(U30-~{E}): track 0.00 -> 2.30 mm
- net Net-(D4-A): track 0.00 -> 1.93 mm
- net Net-(D2-A): track 0.00 -> 1.93 mm
Other:
- board text added: "+5V VDC +3V3"
- board text added: "3V3 GND"
- board text added: "5V GND"
- board text added: "HALL|GND"
- board text added: "Select VDC"

Commit message: Comments
Other:
- board text added: "* Cell Housing: * Mounting hole spacing (X) = 30.5mm * Center = (110.25mm, 125mm) * Rods Dimensions: * Back Side X Vals: [98.75, 104.75, 110.75, 116.75] * Front Side X Vals: [103.75, 109.75, 115.75, 121.75] * magnet_coord_y: 8.7 * motor_shaft_gripper_max_y: 10.3"
- board text removed: "Cell Housing: * Mounting hole spacing (X) = 30.5mm * Center = (110.25mm, 125mm)"
Changed lines of the file:
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@@
 		)
 	)
-	(gr_text "Cell Housing:\n	* Mounting hole spacing (X) = 30.5mm\n	* Center = (110.25mm, 125mm)"
+	(gr_text "* Cell Housing:\n	* Mounting hole spacing (X) = 30.5mm\n	* Center = (110.25mm, 125mm)\n\n* Rods Dimensions:\n	* Back Side X Vals: [98.75, 104.75, 110.75, 116.75]\n	* Front Side X Vals: [103.75, 109.75, 115.75, 121.75]\n	* magnet_coord_y: 8.7\n	* motor_shaft_gripper_max_y: 10.3"
 		(at 192 103.75 0)
 		(layer "Cmts.User")
